File: corne-classic/pcb/corne-classic.kicad_pcb (KiCad board)
At the start: 2 copper layers, 133.8 x 92.2 mm, 98 parts, among them J1 MJ-4PP-9, J2 OLED, J3 LED, P1 i2c-pin, P2 i2c-pin, SW1 SW_PUSH, SW10 SW_PUSH, SW11 SW_PUSH, SW12 SW_PUSH, SW13 SW_PUSH, SW14 SW_PUSH, SW15 SW_PUSH, SW16 SW_PUSH, SW17 SW_PUSH, SW18 SW_PUSH, SW19 SW_PUSH, SW2 SW_PUSH, SW20 SW_PUSH, SW21 SW_PUSH, SW3 SW_PUSH, SW4 SW_PUSH, SW5 SW_PUSH, SW6 SW_PUSH, SW7 SW_PUSH, SW8 SW_PUSH, SW9 SW_PUSH, U1 ProMicro

Commit message: Replaced Arduino by Esp32 TinyS3. Got a crash while rooting ...
Parts:
- removed ? (x9): , kbd:LEGO_HOLE
- removed G*** (x2): LOGO, kbd:corne
- removed U1: ProMicro, kbd:ProMicro_v2
- added TP1: TestPoint, TestPoint:TestPoint_Pad_D1.5mm, B.Cu at (185.8, 127.8)
- added TP2: TestPoint, TestPoint:TestPoint_Pad_D1.5mm, B.Cu at (181.5, 126.3)
- added TP3: TestPoint, TestPoint:TestPoint_Pad_D1.5mm, F.Cu at (185.8, 127.8)
- added TP4: TestPoint, TestPoint:TestPoint_Pad_D1.5mm, F.Cu at (181.5, 126.3)
- added U2: TinyS3_Symbol, easyeda2kicad:TinyS3, F.Cu at (185.7, 85.7)
- added U3: TinyS3_Symbol, easyeda2kicad:TinyS3, B.Cu at (184.6, 87.0)
- RSW1: value Reset -> SW_PUSH
Connections:
- J1 pad B: Net-(J1-PadB) -> Net-(P2-Pin_1)
- L19 pad 1: Net-(L13-Pad1) -> unconnected-(L19-DOUT-Pad1)
- L27 pad 3: Net-(L21-Pad3) -> Net-(L27-DIN)
- P2 pad 1: Net-(J1-PadB) -> Net-(P2-Pin_1)
Routing:
- net LED: track 77.7 -> 18.4 mm, vias 8 -> 4
- net GND: track 797.9 -> 741.0 mm, vias 49 -> 46
- net data: track 55.3 -> 0.10 mm, vias 4 -> 0
- net SDA: track 54.9 -> 0.14 mm, vias 3 -> 0
- net SCL: track 46.4 -> 0.57 mm, vias 2 -> 0
- net reset: track 42.8 -> 0.00 mm, vias 1 -> 0
- net row2: track 215.8 -> 175.3 mm
- net row3: track 121.8 -> 82.9 mm
- net row0: track 205.5 -> 171.5 mm, vias 3 -> 0
- net col1: track 221.3 -> 187.7 mm, vias 4 -> 2
- net col2: track 197.5 -> 165.8 mm, vias 8 -> 6
- net col0: track 245.7 -> 215.0 mm, vias 4 -> 2
- net col3: track 225.1 -> 195.8 mm, vias 6 -> 4
- net col4: track 194.3 -> 167.2 mm, vias 6 -> 4
- net col5: track 187.0 -> 161.8 mm, vias 2 -> 0
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