File: corne-classic/pcb/corne-classic.kicad_pcb (KiCad board)
At the start: 2 copper layers, 133.8 x 92.2 mm, 92 parts, among them J1 MJ-4PP-9, J2 OLED, J3 LED, P1 i2c-pin, P2 i2c-pin, SW1 SW_PUSH, SW10 SW_PUSH, SW11 SW_PUSH, SW12 SW_PUSH, SW13 SW_PUSH, SW14 SW_PUSH, SW15 SW_PUSH, SW16 SW_PUSH, SW17 SW_PUSH, SW18 SW_PUSH, SW19 SW_PUSH, SW2 SW_PUSH, SW20 SW_PUSH, SW21 SW_PUSH, SW3 SW_PUSH, SW4 SW_PUSH, SW5 SW_PUSH, SW6 SW_PUSH, SW7 SW_PUSH, SW8 SW_PUSH, SW9 SW_PUSH, U2 TinyS3_Symbol, U3 TinyS3_Symbol

Commit message: routing + prod files
Parts:
- moved TP1 57.8 mm to (186.7, 70.0)
- moved TP3 57.8 mm to (186.7, 70.0)
- moved TP4 56.4 mm to (182.3, 69.9)
- moved TP2 56.4 mm to (182.2, 69.9)
- moved U3 0.35 mm to (184.2, 87.0)
Connections:
- TP1 pad 1: Net-(U2-VBAT) -> /VBAT
- TP3 pad 1: Net-(U3-VBAT) -> /VBAT
- U2 pad 1: Net-(U2-VBAT) -> /VBAT
- U2 pad 10: col4 -> row3
- U2 pad 11: col5 -> unconnected-(U2-IO0-Pad11)
- U2 pad 16: row3 -> col4
- U2 pad 17: row2 -> col2
- U2 pad 20: row1 -> col1
- U2 pad 21: row0 -> col0
- U2 pad 5: unconnected-(U2-IO1-Pad5) -> row0
- U2 pad 6: col0 -> row1
- U2 pad 7: col1 -> col3
- U2 pad 8: col2 -> col5
- U2 pad 9: col3 -> row2
- U3 pad 1: Net-(U3-VBAT) -> /VBAT
- U3 pad 10: col4 -> row3
- U3 pad 11: col5 -> unconnected-(U3-IO0-Pad11)
- U3 pad 16: row3 -> col4
- U3 pad 17: row2 -> col2
- U3 pad 20: row1 -> col1
- U3 pad 21: row0 -> col0
- U3 pad 5: unconnected-(U3-IO1-Pad5) -> row0
- U3 pad 6: col0 -> row1
- U3 pad 7: col1 -> col3
- U3 pad 8: col2 -> col5
- U3 pad 9: col3 -> row2
Routing:
- net data: track 0.10 -> 58.0 mm, vias 0 -> 1
- net LED: track 18.4 -> 71.9 mm, vias 4 -> 7
- net SDA: track 0.14 -> 49.7 mm
- net SCL: track 0.57 -> 49.9 mm, vias 0 -> 1
- net GND: track 741.0 -> 785.7 mm, vias 46 -> 59
- net row2: track 175.3 -> 213.4 mm
- net row3: track 82.9 -> 119.6 mm
- net VCC: track 734.3 -> 766.3 mm, vias 33 -> 34
- net col3: track 195.8 -> 226.1 mm, vias 4 -> 5
- net col2: track 165.8 -> 196.0 mm
- net reset: track 0.00 -> 28.6 mm, vias 0 -> 2
- net col5: track 161.8 -> 190.0 mm, vias 0 -> 2
- net col4: track 167.2 -> 194.5 mm
- net row0: track 171.5 -> 197.7 mm, vias 0 -> 1
- net col1: track 187.7 -> 213.2 mm
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Other:
- board text added: "+"
- board text added: "-"
